File: SAT_BF.kicad_sch (KiCad schematic)
At the start: 12 parts, among them J1 Screw_Terminal_01x02, U2 ZC323200, U3 module_mpu6050, U4 HMC5883L, U7 INA219, U8 module_bme280

Commit message: troca do RS422 por RS485
Other:
- company: (none) -> SiriusSat-ufma
Changed lines of the file:
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@@
 	(generator_version "9.0")
 	(paper "A4")
+	(title_block
+		(rev "5")
+		(company "SiriusSat-ufma")
+	)
 	(rectangle
 		(start 25.4 100.33)

Commit message: troca de RS422 por RS 485
Parts:
- removed U6: ~, symbol New_Library_MODULE:ESP32_ROCKET
- added J2: Screw_Terminal_01x04, symbol Connector:Screw_Terminal_01x04
Connections:
- net 3V3: now also J2.4 (Pin_4)
- net GND: now also J2.3 (Pin_3)
- net I2C_SCL_2: now also J2.2 (Pin_2)
- net I2C_SDA_2: now also J2.1 (Pin_1)
Changed lines of the file:
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@@
 	)
 	(symbol
-		(lib_id "New_Library_MODULE:ESP32_ROCKET")
-		(at 40.64 46.99 0)
+		(lib_id "Connector:Screw_Terminal_01x04")
+		(at 53.34 52.07 180)
 		(unit 1)
 		(exclude_from_sim no)
@@
 		(dnp no)
 		(fields_autoplaced yes)
-		(property "Reference" "U6"
-			(at 49.53 36.83 0)
+		(property "Reference" "J2"
+			(at 53.34 40.64 0)
 			(effects
 				(font
@@
 			)
 		)
-		(property "Value" "~"
-			(at 49.53 38.1 0)
+		(property "Value" "Screw_Terminal_01x04"
+			(at 53.34 43.18 0)
 			(effects
 				(font
@@
 		)
 		(property "Footprint" ""
-			(at 40.64 46.99 0)
+			(at 53.34 52.07 0)
 			(effects
 				(font
@@
 			)
 		)
-		(property "Datasheet" ""
-			(at 40.64 46.99 0)
+		(property "Datasheet" "~"
+			(at 53.34 52.07 0)
 			(effects
 				(font
@@
 			)
 		)
-		(property "Description" ""
-			(at 40.64 46.99 0)
+		(property "Description" "Generic screw terminal, single row, 01x04, script generated (kicad-library-utils/schlib/autogen/connector/)"
+			(at 53.34 52.07 0)
 			(effects
 				(font
@@
 			)
 		)
-		(pin "1"
+		(pin "4"
 		)
-		(pin "4"
+		(pin "3"
 		)
 		(pin "2"
 		)
-		(pin "3"
+		(pin "1"
 		)
 		(instances
 			(project "SAT_BF"
 				(path "/92b72320-4f9a-43fd-a3c5-8d14c1d8f811"
-					(reference "U6")
+					(reference "J2")
 					(unit 1)
 				)

Commit message: Adicionando Wemmos D1 e atualizando a PCI
Parts:
- added U1: esp32-wemos-d1-mini, esp32-wemos-d1-mini:esp32-wemos-d1-mini, symbol esp32-wemos-d1-mini:esp32-wemos-d1-mini
- U9: value ~ -> esp32_38pins
Changed lines of the file:
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@@
 			)
 		)
-		(property "Value" "~"
+		(property "Value" "esp32_38pins"
 			(at 108.585 27.94 0)
 			(effects
@@
 					(unit 1)
 				)
+			)
+		)
+	)
+	(symbol
+		(lib_id "esp32-wemos-d1-mini:esp32-wemos-d1-mini")
+		(at 209.55 99.06 0)
+		(unit 1)
+		(exclude_from_sim no)
+		(in_bom yes)
+		(on_board yes)
+		(dnp no)
+		(fields_autoplaced yes)
+		(property "Reference" "U1"
+			(at 210.185 95.25 0)
+			(effects
+				(font
+					(size 1.27 1.27)
+				)
+			)
+		)
+		(property "Value" "esp32-wemos-d1-mini"
+			(at 210.185 97.79 0)
+			(effects
+				(font
+					(size 1.27 1.27)
+				)
+			)
+		)
+		(property "Footprint" "esp32-wemos-d1-mini:esp32-wemos-d1-mini"
+			(at 213.36 96.52 0)
+			(effects
+				(font
+					(size 1.27 1.27)
+				)
+				(hide yes)
+			)
+		)
+		(property "Datasheet" ""
+			(at 213.36 96.52 0)
+			(effects
+				(font
+					(size 1.27 1.27)
+				)
+				(hide yes)
+			)
+		)
+		(property "Description" ""
+			(at 209.55 99.06 0)
+			(effects
+				(font
+					(size 1.27 1.27)
+				)
+				(hide yes)
+			)
+		)
+		(pin "9"
+		)
+		(pin "2"
+		)
+		(pin "1"
+		)
+		(pin "5"
+		)
+		(pin "4"
+		)
+		(pin "25"
+		)
+		(pin "8"
+		)
+		(pin "38"
+		)
+		(pin "11"
+		)
+		(pin "34"
+		)
+		(pin "3"
+		)
+		(pin "22"
+		)
+		(pin "6"
+		)
+		(pin "21"
+		)
+		(pin "36"
+		)
+		(pin "7"
+		)
+		(pin "13"
+		)
+		(pin "33"
+		)
+		(pin "10"
+		)
+		(pin "18"
+		)
+		(pin "37"
+		)
+		(pin "23"
+		)
+		(pin "30"
+		)
+		(pin "15"
+		)
+		(pin "24"
+		)
+		(pin "35"
+		)
+		(pin "14"
+		)
+		(pin "28"
+		)
+		(pin "32"
+		)
+		(pin "31"
+		)
+		(pin "29"
+		)
+		(pin "16"
+		)
+		(pin "27"
+		)
+		(pin "40"
+		)
+		(pin "19"
+		)
+		(pin "20"
+		)
+		(pin "39"
+		)
+		(pin "12"
+		)
+		(pin "26"
+		)
+		(pin "17"
+		)
+		(instances
+			(project "SAT_BF"
+				(path "/92b72320-4f9a-43fd-a3c5-8d14c1d8f811"
+					(reference "U1")
+					(unit 1)
+				)

Commit message: atualizações no esquematico
Parts:
- removed U1: esp32-wemos-d1-mini, esp32-wemos-d1-mini:esp32-wemos-d1-mini, symbol esp32-wemos-d1-mini:esp32-wemos-d1-mini
Changed lines of the file:
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@@
-	)
-	(symbol
-		(lib_id "esp32-wemos-d1-mini:esp32-wemos-d1-mini")
-		(at 209.55 99.06 0)
-		(unit 1)
-		(exclude_from_sim no)
-		(in_bom yes)
-		(on_board yes)
-		(dnp no)
-		(fields_autoplaced yes)
-		(property "Reference" "U1"
-			(at 210.185 95.25 0)
-			(effects
-				(font
-					(size 1.27 1.27)
-				)
-			)
-		)
-		(property "Value" "esp32-wemos-d1-mini"
-			(at 210.185 97.79 0)
-			(effects
-				(font
-					(size 1.27 1.27)
-				)
-			)
-		)
-		(property "Footprint" "esp32-wemos-d1-mini:esp32-wemos-d1-mini"
-			(at 213.36 96.52 0)
-			(effects
-				(font
-					(size 1.27 1.27)
-				)
-				(hide yes)
-			)
-		)
-		(property "Datasheet" ""
-			(at 213.36 96.52 0)
-			(effects
-				(font
-					(size 1.27 1.27)
-				)
-				(hide yes)
-			)
-		)
-		(property "Description" ""
-			(at 209.55 99.06 0)
-			(effects
-				(font
-					(size 1.27 1.27)
-				)
-				(hide yes)
-			)
-		)
-		(pin "9"
-		)
-		(pin "2"
-		)
-		(pin "1"
-		)
-		(pin "5"
-		)
-		(pin "4"
-		)
-		(pin "25"
-		)
-		(pin "8"
-		)
-		(pin "38"
-		)
-		(pin "11"
-		)
-		(pin "34"
-		)
-		(pin "3"
-		)
-		(pin "22"
-		)
-		(pin "6"
-		)
-		(pin "21"
-		)
-		(pin "36"
-		)
-		(pin "7"
-		)
-		(pin "13"
-		)
-		(pin "33"
-		)
-		(pin "10"
-		)
-		(pin "18"
-		)
-		(pin "37"
-		)
-		(pin "23"
-		)
-		(pin "30"
-		)
-		(pin "15"
-		)
-		(pin "24"
-		)
-		(pin "35"
-		)
-		(pin "14"
-		)
-		(pin "28"
-		)
-		(pin "32"
-		)
-		(pin "31"
-		)
-		(pin "29"
-		)
-		(pin "16"
-		)
-		(pin "27"
-		)
-		(pin "40"
-		)
-		(pin "19"
-		)
-		(pin "20"
-		)
-		(pin "39"
-		)
-		(pin "12"
-		)
-		(pin "26"
-		)
-		(pin "17"
-		)
-		(instances
-			(project "SAT_BF"
-				(path "/92b72320-4f9a-43fd-a3c5-8d14c1d8f811"
-					(reference "U1")
-					(unit 1)
-				)
-			)
-		)
 	)
 	(symbol

Commit message: trazendo atualizações
Parts:
- added J3: Conn_02x10_Odd_Even, Connector_PinHeader_2.54mm:PinHeader_2x10_P2.54mm_Vertical, symbol Connector_Generic:Conn_02x10_Odd_Even
- added J4: Conn_02x20_Counter_Clockwise, symbol Connector_Generic:Conn_02x20_Counter_Clockwise
- added U1: esp32-wemos-d1-mini, esp32-wemos-d1-mini:esp32-wemos-d1-mini, symbol esp32-wemos-d1-mini:esp32-wemos-d1-mini
Connections:
- net 3V3: now also U1.16 (3V3)
- net CS_SDCARD: now also U1.18 (IO_13/TCK)
- net GND: now also U1.1 (GND), U1.22 (GND), U1.33 (GND)
- net I2C_SCL_1: now also U1.25 (IO_22/D1/SCL)
- net I2C_SCL_2: now also U1.24 (IO_27)
- net I2C_SDA_1: now also U1.27 (IO_21/D2/SDA)
- net LORA_DIO0: now also U1.32 (IO_04)
- net LORA_RST: now also U1.36 (IO_02)
- net NSS_LORA: now also U1.14 (IO_05/D8)
- net RX_GPS: now also U1.29 (IO_17/D3)
- net RX_RS422: now also U1.28 (IO_32)
- net SPI_MISO_1: now also U1.10 (IO_19/D6)
- net SPI_SCK_1: now also U1.8 (IO_18/D5)
- net TX_GPS: now also U1.31 (IO_16/D4)
- net TX_RS422: now also U1.9 (IO_33)
- no-connect marks 36 -> 59

Commit message: adicionando os barramentos
Parts:
- removed J3: Conn_02x10_Odd_Even, Connector_PinHeader_2.54mm:PinHeader_2x10_P2.54mm_Vertical, symbol Connector_Generic:Conn_02x10_Odd_Even
- removed J4: Conn_02x20_Counter_Clockwise, symbol Connector_Generic:Conn_02x20_Counter_Clockwise
- removed U2: ZC323200, ZC323200:XCVR_ZC323200, symbol ZC323200:ZC323200
- removed U9: esp32_38pins, CTE_KICADMOD09_ESP32_38PIN:ESP-32_38PIN, symbol ESP32-38pin:Esp32
Connections:
- net I2C_SDA_2: now also U1.6 (IO_26/D0)
- net SPI_MOSI_1: now also U1.12 (IO_23/D7)
- net RX_GPS: no longer names the net of U1.29 (IO_17/D3)
- net TX_GPS: no longer names the net of U1.31 (IO_16/D4)
- no-connect marks 59 -> 40
Other:
- moved on the sheet: U1
